Commit message: edit urdf loading

File: assets/urdf/arm_hand/arm_hand.urdf (robot description, URDF)
Before this commit: robot xarm7_allegro_hand, 13 links, 12 joints
Links:
- removed link table
- link panda_hand: geometry collision mesh filename=/home/yikai/IsaacGymEnvs/assets/urdf/franka_description/mes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; visual mesh filename=/home/yikai/IsaacGymEnvs/assets/urdf/franka_description/mes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
- link panda_leftfinger: geometry collision mesh filename=/home/yikai/IsaacGymEnvs/assets/factory/mesh/factory_franka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; visual mesh filename=/home/yikai/IsaacGymEnvs/assets/urdf/franka_description/mes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
- link panda_rightfinger: geometry collision mesh filename=/home/yikai/IsaacGymEnvs/assets/factory/mesh/factory_franka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; visual mesh filename=/home/yikai/IsaacGymEnvs/assets/urdf/franka_description/mes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
Joints:
- removed joint table_joint

Commit message: neccesary edit

File: assets/urdf/arm_hand/arm_hand.urdf (robot description, URDF)
Before this commit: robot xarm7_allegro_hand, 12 links, 11 joints
Links:
- link panda_hand: geometry collision mesh filename=../franka_description/meshes/collision/hand.obj; visual mesh filename=../franka_description/meshes/visual/hand.dae
- link panda_leftfinger: geometry collision mesh filename=../../factory/mesh/factory_franka_table/factory_franka_fing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; visual mesh filename=../franka_description/meshes/visual/finger.dae
- link panda_rightfinger: geometry collision mesh filename=../../factory/mesh/factory_franka_table/factory_franka_fing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; visual mesh filename=../franka_description/meshes/visual/finger.dae

Commit message: add hand

File: assets/urdf/arm_hand/arm_hand.urdf (robot description, URDF)
Before this commit: robot xarm7_allegro_hand, 12 links, 11 joints
Links:
- removed link panda_fingertip_centered
- removed link panda_hand
- removed link panda_leftfinger
- removed link panda_rightfinger
- added link link_0.0, mass 0.0119; collision box size=0.0196 0.0275 0.0164; visual mesh filename=meshes/link_0.0.STL
- added link link_1.0, mass 0.065; collision box size=0.0196 0.0275 0.054; visual mesh filename=meshes/link_1.0.STL
- added link link_10.0, mass 0.0355; collision box size=0.0196 0.0275 0.0384; visual mesh filename=meshes/link_2.0.STL
- added link link_11.0, mass 0.0096; collision box size=0.0196 0.0275 0.0267; visual mesh filename=meshes/link_3.0.STL
- added link link_11.0_tip, mass 0.0168; collision sphere radius=0.012; visual mesh filename=meshes/link_3.0_tip.STL
- added link link_12.0, mass 0.0176; collision box size=0.0358 0.034 0.0455; visual mesh filename=meshes/link_12.0_left.STL
- added link link_13.0, mass 0.0119; collision box size=0.0196 0.0275 0.0177; visual mesh filename=meshes/link_13.0.STL
- added link link_14.0, mass 0.038; collision box size=0.0196 0.0275 0.0514; visual mesh filename=meshes/link_14.0.STL
- added link link_15.0, mass 0.0388; collision box size=0.0196 0.0275 0.0423; visual mesh filename=meshes/link_15.0.STL
- added link link_15.0_tip, mass 0.0168; collision sphere radius=0.012; visual mesh filename=meshes/link_15.0_tip.STL
- added link link_2.0, mass 0.0355; collision box size=0.0196 0.0275 0.0384; visual mesh filename=meshes/link_2.0.STL
- added link link_3.0, mass 0.0096; collision box size=0.0196 0.0275 0.0267; visual mesh filename=meshes/link_3.0.STL
- added link link_3.0_tip, mass 0.0168; collision sphere radius=0.012; visual mesh filename=meshes/link_3.0_tip.STL
- added link link_4.0, mass 0.0119; collision box size=0.0196 0.0275 0.0164; visual mesh filename=meshes/link_0.0.STL
- added link link_5.0, mass 0.065; collision box size=0.0196 0.0275 0.054; visual mesh filename=meshes/link_1.0.STL
- added link link_6.0, mass 0.0355; collision box size=0.0196 0.0275 0.0384; visual mesh filename=meshes/link_2.0.STL
- added link link_7.0, mass 0.0096; collision box size=0.0196 0.0275 0.0267; visual mesh filename=meshes/link_3.0.STL
- added link link_7.0_tip, mass 0.0168; collision sphere radius=0.012; visual mesh filename=meshes/link_3.0_tip.STL
- added link link_8.0, mass 0.0119; collision box size=0.0196 0.0275 0.0164; visual mesh filename=meshes/link_0.0.STL
- added link link_9.0, mass 0.065; collision box size=0.0196 0.0275 0.054; visual mesh filename=meshes/link_1.0.STL
- added link palm_link, mass 0.4154; collision box size=0.0408 0.1130 0.095; visual mesh filename=meshes/base_link_left.STL
Joints:
- removed joint panda_finger_joint1
- removed joint panda_finger_joint2
- removed joint panda_fingertip_centered_joint
- removed joint panda_hand_joint
- added joint joint_0.0: type revolute, parent palm_link, child link_0.0, origin xyz=0 -0.0435 -0.001542 rpy=0.08726646255 0 0, axis 0 0 1, limit lower=-0.47 upper=0.47 effort=15 velocity=7
- added joint joint_1.0: type revolute, parent link_0.0, child link_1.0, origin xyz=0 0 0.0164, axis 0 1 0, limit lower=-0.196 upper=1.61 effort=15 velocity=7
- added joint joint_10.0: type revolute, parent link_9.0, child link_10.0, origin xyz=0 0 0.054, axis 0 1 0, limit lower=-0.174 upper=1.709 effort=15 velocity=7
- added joint joint_11.0: type revolute, parent link_10.0, child link_11.0, origin xyz=0 0 0.0384, axis 0 1 0, limit lower=-0.227 upper=1.618 effort=15 velocity=7
- added joint joint_11.0_tip: type fixed, parent link_11.0, child link_11.0_tip, origin xyz=0 0 0.0267 rpy=0 0 0
- added joint joint_12.0: type revolute, parent palm_link, child link_12.0, origin xyz=-0.0182 -0.019333 -0.045987 rpy=0 -1.65806278845 1.5707963259, axis +1 0 0, limit lower=0.263 upper=1.396 effort=15 velocity=7
- added joint joint_13.0: type revolute, parent link_12.0, child link_13.0, origin xyz=-0.027 -0.005 0.0399, axis 0 0 -1, limit lower=-0.105 upper=1.163 effort=15 velocity=7
- added joint joint_14.0: type revolute, parent link_13.0, child link_14.0, origin xyz=0 0 0.0177, axis 0 1 0, limit lower=-0.189 upper=1.644 effort=15 velocity=7
- added joint joint_15.0: type revolute, parent link_14.0, child link_15.0, origin xyz=0 0 0.0514, axis 0 1 0, limit lower=-0.162 upper=1.719 effort=15 velocity=7
- added joint joint_15.0_tip: type fixed, parent link_15.0, child link_15.0_tip, origin xyz=0 0 0.0423 rpy=0 0 0
- added joint joint_2.0: type revolute, parent link_1.0, child link_2.0, origin xyz=0 0 0.054, axis 0 1 0, limit lower=-0.174 upper=1.709 effort=15 velocity=7
- added joint joint_3.0: type revolute, parent link_2.0, child link_3.0, origin xyz=0 0 0.0384, axis 0 1 0, limit lower=-0.227 upper=1.618 effort=15 velocity=7
- added joint joint_3.0_tip: type fixed, parent link_3.0, child link_3.0_tip, origin xyz=0 0 0.0267 rpy=0 0 0
- added joint joint_4.0: type revolute, parent palm_link, child link_4.0, origin xyz=0 0 0.0007 rpy=0.0 0 0, axis 0 0 1, limit lower=-0.47 upper=0.47 effort=15 velocity=7
- added joint joint_5.0: type revolute, parent link_4.0, child link_5.0, origin xyz=0 0 0.0164, axis 0 1 0, limit lower=-0.196 upper=1.61 effort=15 velocity=7
- added joint joint_6.0: type revolute, parent link_5.0, child link_6.0, origin xyz=0 0 0.054, axis 0 1 0, limit lower=-0.174 upper=1.709 effort=15 velocity=7
- added joint joint_7.0: type revolute, parent link_6.0, child link_7.0, origin xyz=0 0 0.0384, axis 0 1 0, limit lower=-0.227 upper=1.618 effort=15 velocity=7
- added joint joint_7.0_tip: type fixed, parent link_7.0, child link_7.0_tip, origin xyz=0 0 0.0267 rpy=0 0 0
- added joint joint_8.0: type revolute, parent palm_link, child link_8.0, origin xyz=0 0.0435 -0.001542 rpy=-0.08726646255 0 0, axis 0 0 1, limit lower=-0.47 upper=0.47 effort=15 velocity=7
- added joint joint_9.0: type revolute, parent link_8.0, child link_9.0, origin xyz=0 0 0.0164, axis 0 1 0, limit lower=-0.196 upper=1.61 effort=15 velocity=7
- added joint joint_hand: type fixed, parent link7, child palm_link, origin xyz=0. 0. 0.095 rpy=0 0 0
